Commit message: Fixed the changes such as the messages not showing and the robot rotates faster as well as it dosen't drift

File: my_rb1_description/urdf/my_rb1_robot.urdf (robot description, URDF)
Before this commit: robot cylinder_robot, 7 links, 6 joints
Links:
- link back_caster: mass 0.25 -> 0.5
- link front_caster: mass 0.25 -> 0.5
- link left_wheel: mass 2.0 -> 1.0; geometry collision cylinder length=0.025 radius=0.025; visual cylinder length=0.025 radius=0.025
- link right_wheel: mass 2.0 -> 1.0; geometry collision cylinder length=0.025 radius=0.025; visual cylinder length=0.025 radius=0.025

Commit message: Third evaluation hopefully everythig is done

File: my_rb1_description/urdf/my_rb1_robot.urdf (robot description, URDF)
Before this commit: robot cylinder_robot, 7 links, 6 joints
Links:
- link back_caster: mass 0.5 -> 0.05
- link front_caster: mass 0.5 -> 0.05
- link right_wheel: geometry collision cylinder length=0.03 radius=0.025; visual cylinder length=0.03 radius=0.025

Commit message: Changed the codes in the urdf file and laser is showing correctly and robot is rotating properly

File: my_rb1_description/urdf/my_rb1_robot.urdf (robot description, URDF)
Before this commit: robot cylinder_robot, 7 links, 6 joints
Links:
- link base_footprint: mass 0.001 -> None; geometry 
- link right_wheel: geometry collision cylinder length=0.025 radius=0.025; visual cylinder length=0.025 radius=0.025
